File: kicad files/hannah_montana.kicad_sch (KiCad schematic)
At the start: 57 parts

Commit message: finished schematic
Parts:
- added SW?: SW_Push, symbol Switch:SW_Push
- added U?: ProMicro, symbol ProMicro:ProMicro
- gave numbers to parts that had none: 1
Connections:
- net GND: now also J?.1 (Pin_1), SW?.1, U?.23 (GND), U?.3 (GND), U?.4 (GND)
- net col0: now also U?.18 (D19/A1(PF6))
- net col1: now also U?.17 (D18/A0(PF7))
- net col2: now also U?.16 (D15/SCLK(PB1))
- net col3: now also U?.15 (D14/MISO(PB3))
- net col4: now also U?.14 (D16/MOSI(PB2))
- net col5: now also U?.13 (D10/A10(PB6))
- net encA: now also U?.20 (D21/A3(PF4))
- net encB: now also U?.19 (D20/A2(PF5))
- net row0: now also U?.7 (D4/A6(PD4))
- net row1: now also U?.8 (D5(PC6))
- net row2: now also U?.9 (D6/A7(PD7))
- net row3: now also U?.10 (D7(PE6))
- net row4: now also U?.11 (D8/A8(PB4))
- net VCC: now reaches J?.2 (Pin_2)
- net VCC: now also U?.21 (VCC)
- net scl: now reaches J?.3 (Pin_3)
- net scl: now also U?.5 (SCL)
- net sda: now reaches J?.4 (Pin_4)
- net sda: now also U?.6 (SDA)
- new net rst: SW?.2, U?.22 (RST)
- no-connect marks 0 -> 4
