File: kicad files/hannah_montana.kicad_pcb (KiCad board)
At the start: 2 copper layers, 59 parts, among them J1 Conn_01x04, SW1 SW_Push, U1 ProMicro

Commit message: placed key footprints
Parts:
- moved MX21 195.3 mm to (42.9, 47.6)
- moved MX20 157.2 mm to (23.8, 47.6)
- moved MX2 152.4 mm to (28.6, 9.53)
- moved MX4 152.0 mm to (66.7, 9.53)
- moved MX1 150.3 mm to (9.53, 9.53)
- moved MX6 143.8 mm to (104.8, 9.53)
- moved MX14 134.0 mm to (71.4, 28.6)
- moved MX12 132.8 mm to (33.3, 28.6)
- moved MX5 131.2 mm to (85.7, 9.53)
- moved MX15 130.6 mm to (90.5, 28.6)
- moved MX8 120.0 mm to (142.9, 9.53)
- moved MX11 118.4 mm to (11.9, 28.6)
- moved MX22 111.9 mm to (61.9, 47.6)
- moved MX13 108.8 mm to (52.4, 28.6)
- moved MX10 105.8 mm to (188.1, 19.1)
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