File: kicad files/_autosave-hannah_montana.kicad_pcb (KiCad board)
At the start: 2 copper layers, 59 parts, among them J1 Conn_01x04, SW1 SW_Push, U1 ProMicro

Commit message: placed diodes
Parts:
- moved D5 142.5 mm to (24.6, 7.94)
- moved D11 137.2 mm to (48.4, 7.94)
- moved D16 130.5 mm to (68.3, 7.94)
- moved D27 122.8 mm to (111.9, 7.94)
- moved D6 122.0 mm to (28.6, 7.94)
- moved D4 116.5 mm to (20.6, 7.94)
- moved D23 115.9 mm to (96.0, 7.94)
- moved D9 114.4 mm to (40.5, 7.94)
- moved D1 111.3 mm to (8.73, 7.94)
- moved D19 109.8 mm to (80.2, 7.94)
- moved D21 108.9 mm to (88.1, 7.94)
- moved D2 108.2 mm to (12.7, 7.94)
- moved D3 105.7 mm to (16.7, 7.94)
- moved D28 105.4 mm to (115.9, 7.94)
- moved D7 102.0 mm to (32.5, 7.94)
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